File: supercar.kicad_sch (KiCad schematic)
At the start: 55 parts, among them U1 74HC283, U2 74HC574, U3 74HC154, U4 74HC574, U5 74HC21, U6 74HC02, U7 74HC04, U8 NE555D

Commit message: Assigned footprints
Parts:
- BT1: footprint (none) -> Battery:BatteryHolder_Keystone_1060_1x2032
- C1, C10, C2, C3, C4, C5, C6, C7, C8, C9: footprint (none) -> Capacitor_SMD:C_1206_3216Metric_Pad1.33x1.80mm_HandSolder
- D1, D10, D11, D12, D13, D14, D15, D16, D2, D3, D4, D5, D6, D7, D8, D9: footprint (none) -> LED_SMD:LED_1206_3216Metric_Pad1.42x1.75mm_HandSolder
- JP1: footprint (none) -> Connector_PinHeader_2.54mm:PinHeader_1x02_P2.54mm_Vertical
- R1, R10, R11, R12, R13, R14, R15, R16, R17, R18, R2, R3, R4, R5, R6, R7, R8, R9: footprint (none) -> Resistor_SMD:R_1206_3216Metric_Pad1.30x1.75mm_HandSolder
- RV1: footprint (none) -> Potentiometer_SMD:Potentiometer_Bourns_3314G_Vertical
- U1: footprint (none) -> Package_SO:SOIC-16_3.9x9.9mm_P1.27mm
- U2, U4: footprint (none) -> Package_SO:SOIC-20W_7.5x12.8mm_P1.27mm
- U3: footprint (none) -> Package_SO:SOIC-24W_7.5x15.4mm_P1.27mm
- U5, U6, U7: footprint (none) -> Package_SO:SOIC-14_3.9x8.7mm_P1.27mm

Commit message: add pcb
Parts:
- JP1: value Power on -> PWR
Connections:
- net at D13.2 (A): now also U3.4 (S3); no longer U3.14 (S12)
- net at D15.2 (A): now also U3.2 (S1); no longer U3.16 (S14)
- net at D16.2 (A): now also U3.1 (S0); no longer U3.17 (S15)
- net at D1.2 (A): now also U3.17 (S15); no longer U3.1 (S0)
- net at D4.2 (A): now also U3.14 (S12); no longer U3.4 (S3)
- net at D3.2 (A): now also U3.15 (S13); no longer U3.3 (S2)
- net at D12.2 (A): now also U3.5 (S4); no longer U3.13 (S11)
- net at D7.2 (A): now also U3.10 (S9); no longer U3.7 (S6)
- net at D9.2 (A): now also U3.8 (S7); no longer U3.9 (S8)
- net at D10.2 (A): now also U3.7 (S6); no longer U3.10 (S9)
- net at U3.11 (S10): now also D6.2 (A); no longer D11.2 (A)
- net at D14.2 (A): now also U3.3 (S2); no longer U3.15 (S13)
- net at D2.2 (A): now also U3.16 (S14); no longer U3.2 (S1)
- net at D5.2 (A): now also U3.13 (S11); no longer U3.5 (S4)
- net at U3.6 (S5): now also D11.2 (A); no longer D6.2 (A)
- net at D8.2 (A): now also U3.9 (S8); no longer U3.8 (S7)
Other:
- moved on the sheet: D1, D10, D11, D12, D13, D14, D15, D16, D2, D3, D4, D5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

Commit message: Carry bit must be set to 0
Connections:
- net GND: now also U1.7 (C0)
- no-connect marks 11 -> 10
Changed lines of the file:
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@@
   (no_connect (at 189.23 125.73))
   (no_connect (at 189.23 130.81))
-  (no_connect (at 111.76 39.37))
   (no_connect (at 187.96 57.15))
   (no_connect (at 187.96 52.07))
@@
     (stroke (width 0) (type default))
   )
+  (wire (pts (xy 109.22 39.37) (xy 109.22 40.64))
+    (stroke (width 0) (type default))
+  )
   (wire (pts (xy 24.13 13.97) (xy 24.13 17.78))
     (stroke (width 0) (type default))
@@
   )
   (wire (pts (xy 271.78 134.62) (xy 274.32 134.62))
+    (stroke (width 0) (type default))
+  )
+  (wire (pts (xy 111.76 39.37) (xy 109.22 39.37))
     (stroke (width 0) (type default))
   )
@@
         )
       )
+    )
+  )
+  (symbol (lib_id "power:GND") (at 109.22 40.64 0) (unit 1)
+    (in_bom yes) (on_board yes) (dnp no)
+    (property "Reference" "#PWR022" (at 109.22 46.99 0)
+      (effects (font (size 1.27 1.27)) hide)
+    )
+    (property "Value" "GND" (at 111.76 41.91 0)
+      (effects (font (size 1.27 1.27)))
+    )
+    (property "Footprint" "" (at 109.22 40.64 0)
+      (effects (font (size 1.27 1.27)) hide)
+    )
+    (property "Datasheet" "" (at 109.22 40.64 0)
+      (effects (font (size 1.27 1.27)) hide)
+    )
+    (pin "1")
+    (instances
+      (project "supercar"
+        (path "/6cdc46ee-6809-405f-bf74-06040b593f5f"
+          (reference "#PWR022") (unit 1)
+        )
+      )

Commit message: Fix led orientation and connection
Connections:
- net +3V3: now also R1.2, R10.2, R11.2, R12.2, R13.2, R14.2, R15.2, R16.2, R2.2, R3.2, R4.2, R5.2, R6.2, R7.2, R8.2, R9.2
- net GND: no longer R1.2, R10.2, R11.2, R12.2, R13.2, R14.2, R15.2, R16.2, R2.2, R3.2, R4.2, R5.2, R6.2, R7.2, R8.2, R9.2
- net at D13.1 (K): now also U3.4 (S3); no longer R13.1
- net at D13.2 (A): now also R13.1; no longer U3.4 (S3)
- net at R3.1: now also D3.2 (A); no longer D3.1 (K)
- net at D15.1 (K): now also U3.2 (S1); no longer R15.1
- net at D15.2 (A): now also R15.1; no longer U3.2 (S1)
- net at R10.1: now also D10.2 (A); no longer D10.1 (K)
- net at R1.1: now also D1.2 (A); no longer D1.1 (K)
- net at D16.1 (K): now also U3.1 (S0); no longer R16.1
- net at D16.2 (A): now also R16.1; no longer U3.1 (S0)
- net at R11.1: now also D11.2 (A); no longer D11.1 (K)
- net at U3.17 (S15): now also D1.1 (K); no longer D1.2 (A)
- net at D4.1 (K): now also U3.14 (S12); no longer R4.1
- net at D4.2 (A): now also R4.1; no longer U3.14 (S12)
- net at R6.1: now also D6.2 (A); no longer D6.1 (K)
- net at U3.15 (S13): now also D3.1 (K); no longer D3.2 (A)
- net at D12.1 (K): now also U3.5 (S4); no longer R12.1
- net at D12.2 (A): now also R12.1; no longer U3.5 (S4)
- net at R2.1: now also D2.2 (A); no longer D2.1 (K)
- net at R7.1: now also D7.2 (A); no longer D7.1 (K)
- net at R5.1: now also D5.2 (A); no longer D5.1 (K)
- net at R8.1: now also D8.2 (A); no longer D8.1 (K)
- net at U3.10 (S9): now also D7.1 (K); no longer D7.2 (A)
- net at D9.1 (K): now also U3.8 (S7); no longer R9.1
- net at D9.2 (A): now also R9.1; no longer U3.8 (S7)
- net at U3.11 (S10): now also D6.1 (K); no longer D6.2 (A)
- net at U3.13 (S11): now also D5.1 (K); no longer D5.2 (A)
- net at U3.16 (S14): now also D2.1 (K); no longer D2.2 (A)
- net at U3.3 (S2): now also D14.1 (K); no longer D14.2 (A)
- net at U3.6 (S5): now also D11.1 (K); no longer D11.2 (A)
- net at U3.7 (S6): now also D10.1 (K); no longer D10.2 (A)
- net at U3.9 (S8): now also D8.1 (K); no longer D8.2 (A)
- net at R14.1: now also D14.2 (A); no longer D14.1 (K)
Other:
- moved on the sheet: D1, D10, D11, D12, D13, D14, D15, D16, D2, D3, D4, D5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
Changed lines of the file:
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@@
   (junction (at 175.26 73.66) (diameter 0) (color 0 0 0 0)
   )
-  (junction (at 266.7 77.47) (diameter 0) (color 0 0 0 0)
-  )
   (junction (at 266.7 62.23) (diameter 0) (color 0 0 0 0)
   )
@@
   (junction (at 39.37 33.02) (diameter 0) (color 0 0 0 0)
   )
+  (junction (at 266.7 39.37) (diameter 0) (color 0 0 0 0)
+  )
   (junction (at 266.7 67.31) (diameter 0) (color 0 0 0 0)
   )
@@
     (stroke (width 0) (type default))
   )
-  (wire (pts (xy 266.7 77.47) (xy 266.7 86.36))
-    (stroke (width 0) (type default))
-  )
   (wire (pts (xy 101.6 168.91) (xy 101.6 171.45))
     (stroke (width 0) (type default))
@@
     (stroke (width 0) (type default))
   )
+  (wire (pts (xy 266.7 33.02) (xy 266.7 39.37))
+    (stroke (width 0) (type default))
+  )
   (wire (pts (xy 271.78 134.62) (xy 274.32 134.62))
     (stroke (width 0) (type default))
@@
     (stroke (width 0) (type default))
   )
-  (wire (pts (xy 266.7 86.36) (xy 222.25 86.36))
-    (stroke (width 0) (type default))
-  )
   (wire (pts (xy 191.77 44.45) (xy 191.77 17.78))
     (stroke (width 0) (type default))
@@
     )
   )
-  (symbol (lib_id "Device:LED") (at 243.84 46.99 0) (mirror y) (unit 1)
+  (symbol (lib_id "Device:LED") (at 243.84 46.99 0) (mirror x) (unit 1)
     (in_bom yes) (on_board yes) (dnp no)
-    (property "Reference" "D13" (at 241.3 48.26 0)
+    (property "Reference" "D13" (at 246.38 45.72 0)
       (effects (font (size 1.27 1.27)))
     )
-    (property "Value" "LED" (at 248.92 48.26 0)
+    (property "Value" "LED" (at 238.76 45.72 0)
       (effects (font (size 1.27 1.27)))
     )
@@
     )
   )
-  (symbol (lib_id "Device:LED") (at 243.84 41.91 0) (mirror y) (unit 1)
+  (symbol (lib_id "Device:LED") (at 243.84 41.91 0) (mirror x) (unit 1)
     (in_bom yes) (on_board yes) (dnp no)
-    (property "Reference" "D15" (at 241.3 43.18 0)
+    (property "Reference" "D15" (at 246.38 40.64 0)
       (effects (font (size 1.27 1.27)))
     )
-    (property "Value" "LED" (at 248.92 43.18 0)
+    (property "Value" "LED" (at 238.76 40.64 0)
       (effects (font (size 1.27 1.27)))
     )
@@
     )
   )
-  (symbol (lib_id "Device:LED") (at 243.84 39.37 0) (mirror y) (unit 1)
+  (symbol (lib_id "Device:LED") (at 243.84 39.37 0) (mirror x) (unit 1)
     (in_bom yes) (on_board yes) (dnp no)
-    (property "Reference" "D16" (at 241.3 40.64 0)
+    (property "Reference" "D16" (at 246.38 38.1 0)
       (effects (font (size 1.27 1.27)))
     )
-    (property "Value" "LED" (at 248.92 40.64 0)
+    (property "Value" "LED" (at 238.76 38.1 0)
       (effects (font (size 1.27 1.27)))
     )
@@
     )
   )
-  (symbol (lib_id "Device:LED") (at 243.84 77.47 0) (mirror y) (unit 1)
+  (symbol (lib_id "power:+3V3") (at 266.7 33.02 0) (unit 1)
+    (in_bom yes) (on_board yes) (dnp no) (fields_autoplaced)
+    (property "Reference" "#PWR023" (at 266.7 36.83 0)
+      (effects (font (size 1.27 1.27)) hide)
+    )
+    (property "Value" "+3V3" (at 266.7 27.94 0)
+      (effects (font (size 1.27 1.27)))
+    )
+    (property "Footprint" "" (at 266.7 33.02 0)
+      (effects (font (size 1.27 1.27)) hide)
+    )
+    (property "Datasheet" "" (at 266.7 33.02 0)
+      (effects (font (size 1.27 1.27)) hide)
+    )
+    (pin "1")
+    (instances
+      (project "supercar"
+        (path "/6cdc46ee-6809-405f-bf74-06040b593f5f"
+          (reference "#PWR023") (unit 1)
+        )
+      )
+    )
+  )
+  (symbol (lib_id "Device:LED") (at 243.84 77.47 0) (mirror x) (unit 1)
     (in_bom yes) (on_board yes) (dnp no)
-    (property "Reference" "D1" (at 241.3 78.74 0)
+    (property "Reference" "D1" (at 246.38 76.2 0)
       (effects (font (size 1.27 1.27)))
     )
-    (property "Value" "LED" (at 248.92 78.74 0)
+    (property "Value" "LED" (at 238.76 76.2 0)
       (effects (font (size 1.27 1.27)))
     )
@@
     )
   )
-  (symbol (lib_id "Device:LED") (at 243.84 69.85 0) (mirror y) (unit 1)
+  (symbol (lib_id "Device:LED") (at 243.84 69.85 0) (mirror x) (unit 1)
     (in_bom yes) (on_board yes) (dnp no)
-    (property "Reference" "D4" (at 241.3 71.12 0)
+    (property "Reference" "D4" (at 246.38 68.58 0)
       (effects (font (size 1.27 1.27)))
     )
-    (property "Value" "LED" (at 248.92 71.12 0)
+    (property "Value" "LED" (at 238.76 68.58 0)
       (effects (font (size 1.27 1.27)))
     )
@@
     )
   )
-  (symbol (lib_id "Device:LED") (at 243.84 72.39 0) (mirror y) (unit 1)
+  (symbol (lib_id "Device:LED") (at 243.84 72.39 0) (mirror x) (unit 1)
     (in_bom yes) (on_board yes) (dnp no)
-    (property "Reference" "D3" (at 241.3 73.66 0)
+    (property "Reference" "D3" (at 246.38 71.12 0)
       (effects (font (size 1.27 1.27)))
     )
-    (property "Value" "LED" (at 248.92 73.66 0)
+    (property "Value" "LED" (at 238.76 71.12 0)
       (effects (font (size 1.27 1.27)))
     )
@@
     )
   )
-  (symbol (lib_id "Device:LED") (at 243.84 49.53 0) (mirror y) (unit 1)
+  (symbol (lib_id "Device:LED") (at 243.84 49.53 0) (mirror x) (unit 1)
     (in_bom yes) (on_board yes) (dnp no)
-    (property "Reference" "D12" (at 241.3 50.8 0)
+    (property "Reference" "D12" (at 246.38 48.26 0)
       (effects (font (size 1.27 1.27)))
     )
-    (property "Value" "LED" (at 248.92 50.8 0)
+    (property "Value" "LED" (at 238.76 48.26 0)
       (effects (font (size 1.27 1.27)))
     )
@@
     )
   )
-  (symbol (lib_id "Device:LED") (at 243.84 62.23 0) (mirror y) (unit 1)
+  (symbol (lib_id "Device:LED") (at 243.84 62.23 0) (mirror x) (unit 1)
     (in_bom yes) (on_board yes) (dnp no)
-    (property "Reference" "D7" (at 241.3 63.5 0)
+    (property "Reference" "D7" (at 246.38 60.96 0)
       (effects (font (size 1.27 1.27)))
     )
-    (property "Value" "LED" (at 248.92 63.5 0)
+    (property "Value" "LED" (at 238.76 60.96 0)
       (effects (font (size 1.27 1.27)))
     )
@@
     )
   )
-  (symbol (lib_id "Device:LED") (at 243.84 57.15 0) (mirror y) (unit 1)
+  (symbol (lib_id "Device:LED") (at 243.84 57.15 0) (mirror x) (unit 1)
     (in_bom yes) (on_board yes) (dnp no)
-    (property "Reference" "D9" (at 241.3 58.42 0)
+    (property "Reference" "D9" (at 246.38 55.88 0)
       (effects (font (size 1.27 1.27)))
     )
-    (property "Value" "LED" (at 248.92 58.42 0)
+    (property "Value" "LED" (at 238.76 55.88 0)
       (effects (font (size 1.27 1.27)))
     )
@@
     )
   )
-  (symbol (lib_id "Device:LED") (at 243.84 59.69 0) (mirror y) (unit 1)
+  (symbol (lib_id "Device:LED") (at 243.84 59.69 0) (mirror x) (unit 1)
     (in_bom yes) (on_board yes) (dnp no)
-    (property "Reference" "D8" (at 241.3 60.96 0)
+    (property "Reference" "D8" (at 246.38 58.42 0)
       (effects (font (size 1.27 1.27)))
     )
-    (property "Value" "LED" (at 248.92 60.96 0)
+    (property "Value" "LED" (at 238.76 58.42 0)
       (effects (font (size 1.27 1.27)))
     )
@@
     )
   )
-  (symbol (lib_id "Device:LED") (at 243.84 67.31 0) (mirror y) (unit 1)
+  (symbol (lib_id "Device:LED") (at 243.84 67.31 0) (mirror x) (unit 1)
     (in_bom yes) (on_board yes) (dnp no)
-    (property "Reference" "D5" (at 241.3 68.58 0)
+    (property "Reference" "D5" (at 246.38 66.04 0)
       (effects (font (size 1.27 1.27)))
     )
-    (property "Value" "LED" (at 248.92 68.58 0)
+    (property "Value" "LED" (at 238.76 66.04 0)
       (effects (font (size 1.27 1.27)))
     )
@@
     )
   )
-  (symbol (lib_id "Device:LED") (at 243.84 44.45 0) (mirror y) (unit 1)
+  (symbol (lib_id "Device:LED") (at 243.84 44.45 0) (mirror x) (unit 1)
     (in_bom yes) (on_board yes) (dnp no)
-    (property "Reference" "D14" (at 241.3 45.72 0)
+    (property "Reference" "D14" (at 246.38 43.18 0)
       (effects (font (size 1.27 1.27)))
     )
-    (property "Value" "LED" (at 248.92 45.72 0)
+    (property "Value" "LED" (at 238.76 43.18 0)
       (effects (font (size 1.27 1.27)))
     )
@@
     )
   )
-  (symbol (lib_id "Device:LED") (at 243.84 74.93 0) (mirror y) (unit 1)
+  (symbol (lib_id "Device:LED") (at 243.84 74.93 0) (mirror x) (unit 1)
     (in_bom yes) (on_board yes) (dnp no)
-    (property "Reference" "D2" (at 241.3 76.2 0)
+    (property "Reference" "D2" (at 246.38 73.66 0)
       (effects (font (size 1.27 1.27)))
     )
-    (property "Value" "LED" (at 248.92 76.2 0)
+    (property "Value" "LED" (at 238.76 73.66 0)
       (effects (font (size 1.27 1.27)))
     )
@@
     )
   )
-  (symbol (lib_id "Device:LED") (at 243.84 52.07 0) (mirror y) (unit 1)
+  (symbol (lib_id "Device:LED") (at 243.84 52.07 0) (mirror x) (unit 1)
     (in_bom yes) (on_board yes) (dnp no)
-    (property "Reference" "D11" (at 241.3 53.34 0)
+    (property "Reference" "D11" (at 246.38 50.8 0)
       (effects (font (size 1.27 1.27)))
     )
-    (property "Value" "LED" (at 248.92 53.34 0)
+    (property "Value" "LED" (at 238.76 50.8 0)
       (effects (font (size 1.27 1.27)))
     )
@@
     )
   )
-  (symbol (lib_id "Device:LED") (at 243.84 54.61 0) (mirror y) (unit 1)
+  (symbol (lib_id "Device:LED") (at 243.84 54.61 0) (mirror x) (unit 1)
     (in_bom yes) (on_board yes) (dnp no)
-    (property "Reference" "D10" (at 241.3 55.88 0)
+    (property "Reference" "D10" (at 246.38 53.34 0)
       (effects (font (size 1.27 1.27)))
     )
-    (property "Value" "LED" (at 248.92 55.88 0)
+    (property "Value" "LED" (at 238.76 53.34 0)
       (effects (font (size 1.27 1.27)))
     )
@@
     )
   )
-  (symbol (lib_id "Device:LED") (at 243.84 64.77 0) (mirror y) (unit 1)
+  (symbol (lib_id "Device:LED") (at 243.84 64.77 0) (mirror x) (unit 1)
     (in_bom yes) (on_board yes) (dnp no)
-    (property "Reference" "D6" (at 241.3 66.04 0)
+    (property "Reference" "D6" (at 246.38 63.5 0)
       (effects (font (size 1.27 1.27)))
     )
-    (property "Value" "LED" (at 248.92 66.04 0)
+    (property "Value" "LED" (at 238.76 63.5 0)
       (effects (font (size 1.27 1.27)))
     )

Commit message: Update the PCB to include a reset circuit
Parts:
- added C11: 1uF, Capacitor_SMD:C_1206_3216Metric_Pad1.33x1.80mm_HandSolder, symbol Device:C_Small
- added D17: 1N4148W, Diode_SMD:D_SOD-123, symbol Diode:1N4148W
- added R19: 100K, Resistor_SMD:R_1206_3216Metric_Pad1.30x1.75mm_HandSolder, symbol Device:R_Small
- added RN1: 10K, Resistor_SMD:R_Array_Convex_4x1206, symbol Device:R_Pack04
Connections:
- net +3V3: now also D17.1 (K), R19.2
- net CLK: now also U8.3 (Q); no longer U7.10
- net GND: now also U7.13, C11.2, RN1.1 (R1.1), RN1.2 (R2.1), RN1.3 (R3.1); no longer U4.1 (OE)
- net at U1.11 (B4), U4.16 (Q3): now also RN1.8 (R1.2)
- net at U1.15 (B3), U4.17 (Q2): now also RN1.7 (R2.2)
- net at U1.2 (B2), U4.18 (Q1): now also RN1.6 (R3.2)
- net at U1.6 (B1), U4.19 (Q0): now also RN1.5 (R4.2)
- net at U7.12: no longer U7.11
- new net: C11.1, D17.2 (A), R19.1, U7.11
- new net +3.3V: RN1.4 (R4.1)
- new net RST: U4.1 (OE), U7.10
- no-connect marks 10 -> 11
Other:
- moved on the sheet: U7E, U7F

Commit message: Reorganize silkscreen a bit
Parts:
- BT1: value Battery_Cell -> CR2032
Changed lines of the file:
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@@
       (effects (font (size 1.27 1.27)) (justify left))
     )
-    (property "Value" "Battery_Cell" (at 105.41 165.7985 0)
+    (property "Value" "CR2032" (at 105.41 165.7985 0)
       (effects (font (size 1.27 1.27)) (justify left))
     )

Commit message: Update schematic and PCB
Parts:
- removed JP1: PWR, Connector_PinHeader_2.54mm:PinHeader_1x02_P2.54mm_Vertical, symbol Jumper:Jumper_2_Open
- added SW1: Power, Button_Switch_THT:SW_Slide_1P2T_CK_OS102011MS2Q, symbol Switch:SW_SPDT
Connections:
- net +3V3: now also SW1.2 (B)
- net at BT1.1 (+): now also SW1.1 (A)
- no-connect marks 11 -> 12
Changed lines of the file:
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@@
   (no_connect (at 187.96 52.07))
   (no_connect (at 189.23 128.27))
+  (no_connect (at 95.25 163.83))
   (no_connect (at 137.16 52.07))
   (no_connect (at 80.01 25.4))
@@
     (stroke (width 0) (type default))
   )
-  (wire (pts (xy 90.17 158.75) (xy 86.36 158.75))
+  (wire (pts (xy 85.09 161.29) (xy 81.28 161.29))
     (stroke (width 0) (type default))
   )
@@
     (stroke (width 0) (type default))
   )
-  (wire (pts (xy 100.33 158.75) (xy 101.6 158.75))
-    (stroke (width 0) (type default))
-  )
   (wire (pts (xy 214.63 107.95) (xy 214.63 110.49))
     (stroke (width 0) (type default))
@@
     (stroke (width 0) (type default))
   )
+  (wire (pts (xy 95.25 158.75) (xy 101.6 158.75))
+    (stroke (width 0) (type default))
+  )
   (wire (pts (xy 86.36 44.45) (xy 86.36 121.92))
     (stroke (width 0) (type default))
@@
     (stroke (width 0) (type default))
   )
-  (wire (pts (xy 86.36 156.21) (xy 86.36 158.75))
+  (wire (pts (xy 81.28 158.75) (xy 81.28 161.29))
     (stroke (width 0) (type default))
   )
@@
     )
   )
-  (symbol (lib_id "Jumper:Jumper_2_Open") (at 95.25 158.75 0) (unit 1)
-    (in_bom yes) (on_board yes) (dnp no) (fields_autoplaced)
-    (property "Reference" "JP1" (at 95.25 152.4 0)
-      (effects (font (size 1.27 1.27)))
-    )
-    (property "Value" "PWR" (at 95.25 154.94 0)
-      (effects (font (size 1.27 1.27)))
-    )
-    (property "Footprint" "Connector_PinHeader_2.54mm:PinHeader_1x02_P2.54mm_Vertical" (at 95.25 158.75 0)
-      (effects (font (size 1.27 1.27)) hide)
-    )
-    (property "Datasheet" "~" (at 95.25 158.75 0)
-      (effects (font (size 1.27 1.27)) hide)
-    )
-    (pin "2")
-    (pin "1")
-    (instances
-      (project "supercar"
-        (path "/6cdc46ee-6809-405f-bf74-06040b593f5f"
-          (reference "JP1") (unit 1)
-        )
-      )
-    )
-  )
   (symbol (lib_id "Device:R_Small") (at 255.27 62.23 90) (mirror x) (unit 1)
     (in_bom yes) (on_board yes) (dnp no)
@@
     )
   )
-  (symbol (lib_id "power:+3V3") (at 86.36 156.21 0) (unit 1)
+  (symbol (lib_id "power:+3V3") (at 81.28 158.75 0) (unit 1)
     (in_bom yes) (on_board yes) (dnp no) (fields_autoplaced)
-    (property "Reference" "#PWR020" (at 86.36 160.02 0)
+    (property "Reference" "#PWR020" (at 81.28 162.56 0)
       (effects (font (size 1.27 1.27)) hide)
     )
-    (property "Value" "+3V3" (at 86.36 151.13 0)
+    (property "Value" "+3V3" (at 81.28 153.67 0)
       (effects (font (size 1.27 1.27)))
     )
-    (property "Footprint" "" (at 86.36 156.21 0)
+    (property "Footprint" "" (at 81.28 158.75 0)
       (effects (font (size 1.27 1.27)) hide)
     )
-    (property "Datasheet" "" (at 86.36 156.21 0)
+    (property "Datasheet" "" (at 81.28 158.75 0)
       (effects (font (size 1.27 1.27)) hide)
     )
@@
         )
       )
+    )
+  )
+  (symbol (lib_id "Switch:SW_SPDT") (at 90.17 161.29 0) (unit 1)
+    (in_bom yes) (on_board yes) (dnp no) (fields_autoplaced)
+    (property "Reference" "SW1" (at 90.17 152.4 0)
+      (effects (font (size 1.27 1.27)))
+    )
+    (property "Value" "Power" (at 90.17 154.94 0)
+      (effects (font (size 1.27 1.27)))
+    )
+    (property "Footprint" "Button_Switch_THT:SW_Slide_1P2T_CK_OS102011MS2Q" (at 90.17 161.29 0)
+      (effects (font (size 1.27 1.27)) hide)
+    )
+    (property "Datasheet" "~" (at 90.17 168.91 0)
+      (effects (font (size 1.27 1.27)) hide)
+    )
+    (pin "2")
+    (pin "1")
+    (pin "3")
+    (instances
+      (project "supercar"
+        (path "/6cdc46ee-6809-405f-bf74-06040b593f5f"
+          (reference "SW1") (unit 1)
+        )
+      )
